File: boardswap.kicad_pcb (KiCad board)
At the start: 2 copper layers, 285 x 93.7 mm, 161 parts, among them J1 USB_C_Receptacle_USB2.0, SW1 SW_Push, U1 ATmega32U4-AU, U2 USBLC6-2SC6, Y1 16MHz

Commit message: final version, might add flex cuts later
Parts:
- moved D28 13.6 mm to (270.5, 78.4)
- moved D3 7.78 mm to (52.4, 53.6), turned to 90 degrees
- moved D15 7.78 mm to (9.53, 72.6), turned to 90 degrees
- moved D24 7.68 mm to (185.7, 73.1), turned to 90 degrees
- moved D42 7.66 mm to (266.7, 92.1), turned to 90 degrees
- moved D68 7.66 mm to (266.7, 130.2), turned to 90 degrees
- moved D13 7.66 mm to (242.9, 54.0), turned to 90 degrees
- moved D41 7.66 mm to (242.9, 92.1), turned to 90 degrees
- moved D55 7.66 mm to (242.9, 111.2), turned to 90 degrees
- moved D27 7.66 mm to (242.9, 73.1), turned to 90 degrees
- moved D67 7.66 mm to (242.9, 130.2), turned to 90 degrees
- moved D56 7.66 mm to (266.7, 111.2), turned to 90 degrees
- moved D12 7.66 mm to (223.8, 54.0), turned to 90 degrees
- moved D40 7.66 mm to (223.8, 92.1), turned to 90 degrees
- moved D14 7.66 mm to (266.7, 54.0), turned to 90 degrees
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Routing:
- net ROW3: track 302.6 -> 283.7 mm
- net Net-(D44-Pad2): track 39.6 -> 20.9 mm, vias 4 -> 2
- net ROW0: track 387.8 -> 372.1 mm, vias 17 -> 16
- net COL1: track 89.5 -> 102.3 mm
- net ROW2: track 311.8 -> 302.6 mm, vias 18 -> 17
- net ROW4: track 312.8 -> 306.0 mm, vias 14 -> 15
- net Net-(D15-Pad2): track 10.2 -> 3.36 mm
- net Net-(D3-Pad2): track 10.2 -> 3.50 mm
- net Net-(D55-Pad2): track 10.2 -> 3.96 mm
- net Net-(D11-Pad2): track 10.2 -> 3.96 mm
- net Net-(D21-Pad2): track 10.2 -> 3.96 mm
- net Net-(D18-Pad2): track 10.2 -> 3.96 mm
- net Net-(D56-Pad2): track 10.2 -> 3.96 mm
- net Net-(D38-Pad2): track 10.2 -> 3.96 mm
- net Net-(D26-Pad2): track 10.2 -> 3.96 mm
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Other:
- board size 285 x 93.7 mm -> 285 x 95.1 mm
